Commit message: feat: elevator (ArrowUp/Down) and gripper (G/B) control with linkage coupling

File: TR4_Pro/TR4_with_grippers_v2.urdf (robot description, URDF)
Before this commit: robot TR4, 30 links, 29 joints
Joints:
- joint elevation: limit lower=0 upper=0 effort=0 velocity=0 -> lower=0 upper=0.35 effort=0 velocity=0

Commit message: fix: elevator limits (0-0.8), init=0.3, cache-bust URDF URL

File: TR4_Pro/TR4_with_grippers_v2.urdf (robot description, URDF)
Before this commit: robot TR4, 30 links, 29 joints
Joints:
- joint elevation: limit lower=0 upper=0.35 effort=0 velocity=0 -> lower=0 upper=0.8 effort=0 velocity=0

Commit message: fix: elevator limits (-0.8~0), gripper joint3 counter-rotation, arm switch jump

File: TR4_Pro/TR4_with_grippers_v2.urdf (robot description, URDF)
Before this commit: robot TR4, 30 links, 29 joints
Joints:
- joint elevation: limit lower=0 upper=0.8 effort=0 velocity=0 -> lower=-0.8 upper=0 effort=0 velocity=0

Commit message: fix: gripper open/closed positions from calibration, expand joint2 limits to ±1.0472

File: TR4_Pro/TR4_with_grippers_v2.urdf (robot description, URDF)
Before this commit: robot TR4, 30 links, 29 joints
Joints:
- joint left_gripper_l_joint2: limit lower=-1.0472 upper=0 effort=0 velocity=0 -> lower=-1.0472 upper=1.0472 effort=0 velocity=0
- joint left_gripper_r_joint2: limit lower=0 upper=1.0472 effort=0 velocity=0 -> lower=-1.0472 upper=1.0472 effort=0 velocity=0
- joint right_gripper_l_joint2: limit lower=-1.0472 upper=0 effort=0 velocity=0 -> lower=-1.0472 upper=1.0472 effort=0 velocity=0
- joint right_gripper_r_joint2: limit lower=0 upper=1.0472 effort=0 velocity=0 -> lower=-1.0472 upper=1.0472 effort=0 velocity=0
